File: CertusNX.kicad_pcb (KiCad board)
At the start: 2 copper layers, 144 parts, among them J1 USB_C_Receptacle, J2 Conn_01x06, J3 RJLD260TC1, J4 RJLD260TC1, J5 Conn_02x10_Odd_Even, J6 Conn_02x10_Odd_Even, SW1 SW_Push, SW2 SW_SPDT, U1 LFD2NX-17-7MG121I, U10 DP83822, U2 FT232H, U3 W25Q128JVP, U4 FSUSB42MUX, U5 DP83822, U6 TLV62569ADRL, U7 TLV62569ADRL, U8 TLV62569ADRL, U9 TPSM53604RDA, Y1 SiT8008xx-7x-xxN

Commit message: 配置(あきらめ)
Parts:
- removed C49, C57: 0.1u, Passive_Robotech:1608-C
- removed C50, C51: 0.01u, Passive_Robotech:1608-C
- removed C55: 22n, Passive_Robotech:1608-C
- removed C58: 10u, Passive_Robotech:2012-C
- removed FB7: 120Ohm, Inductor_SMD:L_0603_1608Metric_Pad1.05x0.95mm_HandSolder
- removed J6: Conn_02x10_Odd_Even, Connector_Molex:Molex_SlimStack_52991-0208_2x10_P0.50mm_Vertical
- removed R21: 10k, Passive_Robotech:2012-R
- removed R34: 1.96k, Passive_Robotech:2012-R
- removed R35: 2.49k, Passive_Robotech:2012-R
- removed R36: 4.87k, Passive_Robotech:2012-R
- removed R37, R38, R39, R40: 49.9, Passive_Robotech:2012-R
- removed R51: 2.2k, Passive_Robotech:2012-R
- removed U5: DP83822, IC_Robotech:DP83822
- added L1: 2.2uH, Inductor_SMD:L_1210_3225Metric_Pad1.42x2.65mm_HandSolder, F.Cu at (104.6, 119.1)
- added L2: 2.2uH, Inductor_SMD:L_1210_3225Metric_Pad1.42x2.65mm_HandSolder, F.Cu at (97.1, 119.1)
- added L3: 2.2uH, Inductor_SMD:L_1210_3225Metric_Pad1.42x2.65mm_HandSolder, F.Cu at (108.0, 141.7)
- C12, C14, C18, C23, C26, D7, FB1, FB2, FB3: moved to B.Cu
- C52, C53, C54, C67: footprint Passive_Robotech:1608-C -> Capacitor_SMD:C_0402_1005Metric_Pad0.74x0.62mm_HandSolder
- C59, C60, C61, C62, C63, C64, C65, C66: footprint Passive_Robotech:2012-C -> Capacitor_SMD:C_0603_1608Metric_Pad1.08x0.95mm_HandSolder
- J1: value USB_C_Receptacle -> Conn_02x30_Odd_Even; footprint Connector_USB:USB_C_Receptacle_Molex_105450-0101 -> Connector_Molex:Molex_SlimStack_52991-0608_2x30_P0.50mm_Vertical; moved to B.Cu
- J3: value RJLD260TC1 -> USB_C_Receptacle_USB2.0_16P; footprint Connector_Robotech:RJLD260TC1 -> Connector_USB:USB_C_Receptacle_GCT_USB4105-xx-A_16P_TopMnt_Horizontal
- J5: value Conn_02x10_Odd_Even -> Conn_02x30_Odd_Even; footprint Connector_Molex:Molex_SlimStack_52991-0208_2x10_P0.50mm_Vertical -> Connector_Molex:Molex_SlimStack_52991-0608_2x30_P0.50mm_Vertical; moved to B.Cu
- R44, R45, R46, R47, R52: footprint Passive_Robotech:2012-R -> Resistor_SMD:R_0402_1005Metric_Pad0.72x0.64mm_HandSolder
- U2: footprint Package_QFP:LQFP-48_7x7mm_P0.5mm -> Package_DFN_QFN:QFN-48-1EP_8x8mm_P0.5mm_EP6.2x6.2mm
- U4: footprint Package_SO:MSOP-10_3x3mm_P0.5mm -> Local:FSUSB42UMX
- moved J5 71.8 mm to (115.5, 109.5)
- moved R20 63.2 mm to (123.1, 140.1), turned to 180 degrees
- moved D5 61.9 mm to (128.2, 136.1)
- moved R28 61.8 mm to (125.6, 136.1)
- moved D6 61.1 mm to (128.2, 137.3)
- moved R29 61.1 mm to (125.6, 137.3)
- moved D2 59.2 mm to (128.2, 133.7)
- moved R17 59.2 mm to (125.6, 133.7)
- moved D1 58.7 mm to (128.2, 131.3)
- moved R16 58.7 mm to (125.6, 131.3)
- moved SW1 58.2 mm to (127.0, 140.1), turned to 180 degrees
- moved LED1 57.2 mm to (127.8, 128.8)
- moved D4 57.0 mm to (128.2, 134.9)
- moved R19 57.0 mm to (125.6, 134.9)
- moved R31 57.0 mm to (107.2, 130.1), turned to 90 degrees
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Connections:
- R22 pad 1: Net-(J1-D--PadA7) -> Net-(J3-D--PadA7)
- R23 pad 1: Net-(J1-D+-PadA6) -> Net-(J3-D+-PadA6)
- R24 pad 1: Net-(J1-CC1) -> Net-(J3-CC1)
- R25 pad 1: Net-(J1-CC2) -> Net-(J3-CC2)
Routing:
- net GND: track 0.00 -> 14.9 mm, vias 0 -> 28
- net +3V3: track 0.00 -> 8.02 mm
- net +5V: track 0.00 -> 7.12 mm
- net Net-(U2-XCSI): track 0.00 -> 4.88 mm
- net +1V8: track 0.00 -> 4.47 mm, vias 0 -> 2
- net Net-(J3-D--PadA7): track 0.00 -> 4.34 mm
- net Net-(J3-D+-PadA6): track 0.00 -> 3.35 mm
- net Net-(U2-VPLL): track 0.00 -> 3.10 mm
- net Net-(U9-FB): track 0.00 -> 3.09 mm
- net Net-(U2-VPHY): track 0.00 -> 3.06 mm
- net Net-(U2-~{RESET}): track 0.00 -> 2.96 mm
- net Net-(U7-FB): track 0.00 -> 2.75 mm
- net Net-(U6-FB): track 0.00 -> 2.75 mm
- net Net-(U8-FB): track 0.00 -> 2.75 mm
- net Net-(U2-VCCA): track 0.00 -> 1.93 mm
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- added copper zone on F.Cu, net +12V
- added copper zone on F.Cu, net +1V
- added copper zone on F.Cu, net +1V8
- added copper zone on F.Cu, net +3V3
- added copper zone on F.Cu, net +5V
- added copper zone on F.Cu, net Net-(U6-SW)
- added copper zone on F.Cu, net Net-(U7-SW)
- added copper zone on F.Cu, net Net-(U8-SW)
Other:
- board outline added: 40 x 40 mm
- copper layers 2 -> 4

Commit message: pin仮
Parts:
- C11, C13, C14, C16, C19, C20, C21, C22, C24, C25, C27, C28, C29, C33, C47: footprint Capacitor_SMD:C_0402_1005Metric_Pad0.74x0.62mm_HandSolder -> Capacitor_SMD:C_0201_0603Metric
- C15, C17: moved to B.Cu
- J1, J5: value Conn_02x30_Odd_Even -> Conn_02x20_Odd_Even; footprint Connector_Molex:Molex_SlimStack_52991-0608_2x30_P0.50mm_Vertical -> Connector_Molex:Molex_SlimStack_52991-0408_2x20_P0.50mm_Vertical
- moved C48 29.7 mm to (139.6, 132.6)
- moved R10 29.7 mm to (137.6, 131.4)
- moved R7 29.7 mm to (137.6, 132.7)
- moved C26 13.4 mm to (105.8, 132.4), turned to -90 degrees
- moved FB3 12.6 mm to (115.2, 133.7), turned to 90 degrees
- moved FB2 12.2 mm to (105.8, 128.4)
- moved R30 12.1 mm to (116.2, 133.2), turned to 90 degrees
- moved C25 11.0 mm to (107.7, 133.2), turned to -90 degrees
- moved C23 10.8 mm to (113.6, 133.8), turned to -90 degrees
- moved R32 10.2 mm to (115.0, 133.2), turned to -90 degrees
- moved C27 9.78 mm to (107.7, 131.7), turned to -90 degrees
- moved C28 9.65 mm to (107.2, 129.2), turned to 90 degrees
- moved C13 9.38 mm to (110.2, 133.2), turned to -90 degrees
- moved C18 9.25 mm to (108.5, 127.0), turned to 0 degrees
- moved C24 8.81 mm to (111.4, 133.4), turned to 0 degrees
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Connections:
- J1 pad 1: unconnected-(J1-Pin_1-Pad1) -> GND
- J1 pad 10: unconnected-(J1-Pin_10-Pad10) -> PB46B_L11
- J1 pad 11: unconnected-(J1-Pin_11-Pad11) -> PB40A_K10
- J1 pad 12: unconnected-(J1-Pin_12-Pad12) -> PB40B_K11
- J1 pad 13: unconnected-(J1-Pin_13-Pad13) -> PB42A_J8
- J1 pad 14: unconnected-(J1-Pin_14-Pad14) -> PB42B_J7
- J1 pad 15: unconnected-(J1-Pin_15-Pad15) -> PB48A_J10
- J1 pad 16: unconnected-(J1-Pin_16-Pad16) -> PB48B_J11
- J1 pad 17: unconnected-(J1-Pin_17-Pad17) -> PB44A_H11
- J1 pad 18: unconnected-(J1-Pin_18-Pad18) -> PB44B_H10
- J1 pad 19: unconnected-(J1-Pin_19-Pad19) -> PB54A_G9
- J1 pad 2: unconnected-(J1-Pin_2-Pad2) -> GND
- J1 pad 20: unconnected-(J1-Pin_20-Pad20) -> PB54B_G8
- J1 pad 21: unconnected-(J1-Pin_21-Pad21) -> PB22A_H7
- J1 pad 22: unconnected-(J1-Pin_22-Pad22) -> PB22B_G7
- J1 pad 23: unconnected-(J1-Pin_23-Pad23) -> PB20A_G10
- J1 pad 24: unconnected-(J1-Pin_24-Pad24) -> PB20B_G11
- J1 pad 25: unconnected-(J1-Pin_25-Pad25) -> PB26A_F8
- J1 pad 26: unconnected-(J1-Pin_26-Pad26) -> PB26B_F9
- J1 pad 27: unconnected-(J1-Pin_27-Pad27) -> PR30A_E7
- J1 pad 28: unconnected-(J1-Pin_28-Pad28) -> PB30B_F7
- J1 pad 3: unconnected-(J1-Pin_3-Pad3) -> PB56A_K7
- J1 pad 30: unconnected-(J1-Pin_30-Pad30) -> PR65B_D8
- J1 pad 31: unconnected-(J1-Pin_31-Pad31) -> PB18A_F11
- J1 pad 32: unconnected-(J1-Pin_32-Pad32) -> PB18B_F10
- J1 pad 33: unconnected-(J1-Pin_33-Pad33) -> PB16A_E11
- J1 pad 34: unconnected-(J1-Pin_34-Pad34) -> PB16B_E10
- J1 pad 39: unconnected-(J1-Pin_39-Pad39) -> GND
- J1 pad 4: unconnected-(J1-Pin_4-Pad4) -> PB56B_L7
- J1 pad 40: unconnected-(J1-Pin_40-Pad40) -> GND
- J1 pad 5: unconnected-(J1-Pin_5-Pad5) -> PB52A_L8
- J1 pad 6: unconnected-(J1-Pin_6-Pad6) -> PB52B_K8
- J1 pad 7: unconnected-(J1-Pin_7-Pad7) -> PB50A_L9
- J1 pad 8: unconnected-(J1-Pin_8-Pad8) -> PB50B_K9
- J1 pad 9: unconnected-(J1-Pin_9-Pad9) -> PB46A_L10
- J5 pad 1: unconnected-(J5-Pin_1-Pad1) -> GND
- J5 pad 10: unconnected-(J5-Pin_10-Pad10) -> +5V
- J5 pad 11: unconnected-(J5-Pin_11-Pad11) -> PB70A_L2
- J5 pad 12: unconnected-(J5-Pin_12-Pad12) -> PB70B_L1
- J5 pad 13: unconnected-(J5-Pin_13-Pad13) -> PB62A_L5
- J5 pad 14: unconnected-(J5-Pin_14-Pad14) -> PB62B_L6
- J5 pad 15: unconnected-(J5-Pin_15-Pad15) -> PB64A_J5
- J5 pad 16: unconnected-(J5-Pin_16-Pad16) -> PB64B_K4
- J5 pad 17: unconnected-(J5-Pin_17-Pad17) -> PB68A_J1
- J5 pad 18: unconnected-(J5-Pin_18-Pad18) -> PB68B_J2
- J5 pad 19: unconnected-(J5-Pin_19-Pad19) -> PB66A_H4
- J5 pad 2: unconnected-(J5-Pin_2-Pad2) -> GND
- J5 pad 20: unconnected-(J5-Pin_20-Pad20) -> PB66B_J4
- J5 pad 21: unconnected-(J5-Pin_21-Pad21) -> PB60A_G5
- J5 pad 22: unconnected-(J5-Pin_22-Pad22) -> PB60B_H5
- J5 pad 23: unconnected-(J5-Pin_23-Pad23) -> PB58A_K5
- J5 pad 24: unconnected-(J5-Pin_24-Pad24) -> PB58B_K6
- J5 pad 25: unconnected-(J5-Pin_25-Pad25) -> PB24A_F6
- J5 pad 26: unconnected-(J5-Pin_26-Pad26) -> PB24B_F5
- J5 pad 27: unconnected-(J5-Pin_27-Pad27) -> PR28A_E6
- J5 pad 28: unconnected-(J5-Pin_28-Pad28) -> PR28B_E5
- J5 pad 29: unconnected-(J5-Pin_29-Pad29) -> PT67A_B3
- J5 pad 3: unconnected-(J5-Pin_3-Pad3) -> +1V
- J5 pad 30: unconnected-(J5-Pin_30-Pad30) -> PT67B_C3
- J5 pad 31: unconnected-(J5-Pin_31-Pad31) -> PR13A_E3
- J5 pad 32: unconnected-(J5-Pin_32-Pad32) -> PR13B_F1
- J5 pad 33: unconnected-(J5-Pin_33-Pad33) -> PR11A_E2
- J5 pad 34: unconnected-(J5-Pin_34-Pad34) -> PR11B_E1
- J5 pad 36: unconnected-(J5-Pin_36-Pad36) -> PR9B_D1
- J5 pad 37: unconnected-(J5-Pin_37-Pad37) -> PR7A_B2
- J5 pad 38: unconnected-(J5-Pin_38-Pad38) -> PR7B_C2
- J5 pad 39: unconnected-(J5-Pin_39-Pad39) -> GND
- J5 pad 4: unconnected-(J5-Pin_4-Pad4) -> +1V
- J5 pad 40: unconnected-(J5-Pin_40-Pad40) -> GND
- J5 pad 5: unconnected-(J5-Pin_5-Pad5) -> +1V8
- J5 pad 6: unconnected-(J5-Pin_6-Pad6) -> +1V8
- J5 pad 7: unconnected-(J5-Pin_7-Pad7) -> +3V3
- J5 pad 8: unconnected-(J5-Pin_8-Pad8) -> +3V3
- J5 pad 9: unconnected-(J5-Pin_9-Pad9) -> +5V
- U1 pad B2: unconnected-(U1A-PR7A-PadB2) -> PR7A_B2
- U1 pad B3: unconnected-(U1A-PT67A-PadB3) -> PT67A_B3
- U1 pad C2: unconnected-(U1A-PR7B-PadC2) -> PR7B_C2
- U1 pad C3: unconnected-(U1A-PT67B-PadC3) -> PT67B_C3
- U1 pad D1: unconnected-(U1A-PR9B-PadD1) -> PR9B_D1
- U1 pad D8: unconnected-(U1A-PT65B-PadD8) -> PR65B_D8
- U1 pad E1: unconnected-(U1A-PR11B-PadE1) -> PR11B_E1
- U1 pad E10: unconnected-(U1B-PB16B-PadE10) -> PB16B_E10
- U1 pad E11: unconnected-(U1B-PB16A-PadE11) -> PB16A_E11
- U1 pad E2: unconnected-(U1A-PR11A-PadE2) -> PR11A_E2
- U1 pad E3: unconnected-(U1A-PR13A-PadE3) -> PR13A_E3
- U1 pad E5: unconnected-(U1A-PB28B-PadE5) -> PR28B_E5
- U1 pad E6: unconnected-(U1A-PB28A-PadE6) -> PR28A_E6
- U1 pad E7: unconnected-(U1A-PB30A-PadE7) -> PR30A_E7
- U1 pad F1: unconnected-(U1A-PR13B-PadF1) -> PR13B_F1
- U1 pad F10: unconnected-(U1B-PB18B-PadF10) -> PB18B_F10
- U1 pad F11: unconnected-(U1B-PB18A-PadF11) -> PB18A_F11
- U1 pad F5: unconnected-(U1A-PB24B-PadF5) -> PB24B_F5
- U1 pad F6: unconnected-(U1A-PB24A-PadF6) -> PB24A_F6
- U1 pad F7: unconnected-(U1A-PB30B-PadF7) -> PB30B_F7
- U1 pad F8: unconnected-(U1A-PB26A-PadF8) -> PB26A_F8
- U1 pad F9: unconnected-(U1A-PB26B-PadF9) -> PB26B_F9
- U1 pad G10: unconnected-(U1B-PB20A-PadG10) -> PB20A_G10
- U1 pad G11: unconnected-(U1B-PB20B-PadG11) -> PB20B_G11
- U1 pad G5: unconnected-(U1A-PB60A-PadG5) -> PB60A_G5
- U1 pad G7: unconnected-(U1A-PB22B-PadG7) -> PB22B_G7
- U1 pad G8: unconnected-(U1B-PB54B-PadG8) -> PB54B_G8
- U1 pad G9: unconnected-(U1B-PB54A-PadG9) -> PB54A_G9
- U1 pad H10: unconnected-(U1B-PB44B-PadH10) -> PB44B_H10
- U1 pad H11: unconnected-(U1B-PB44A-PadH11) -> PB44A_H11
- U1 pad H4: unconnected-(U1B-PB66A-PadH4) -> PB66A_H4
- U1 pad H5: unconnected-(U1B-PB60B-PadH5) -> PB60B_H5
- U1 pad H7: unconnected-(U1B-PB22A-PadH7) -> PB22A_H7
- U1 pad J1: unconnected-(U1B-PB68A-PadJ1) -> PB68A_J1
- U1 pad J10: unconnected-(U1B-PB48A-PadJ10) -> PB48A_J10
- U1 pad J11: unconnected-(U1B-PB48B-PadJ11) -> PB48B_J11
- U1 pad J2: unconnected-(U1B-PB68B-PadJ2) -> PB68B_J2
- U1 pad J4: unconnected-(U1B-PB66B-PadJ4) -> PB66B_J4
- U1 pad J5: unconnected-(U1B-PB64A-PadJ5) -> PB64A_J5
- U1 pad J7: unconnected-(U1B-PB42B-PadJ7) -> PB42B_J7
- U1 pad J8: unconnected-(U1B-PB42A-PadJ8) -> PB42A_J8
- U1 pad K10: unconnected-(U1B-PB40A-PadK10) -> PB40A_K10
- U1 pad K11: unconnected-(U1B-PB40B-PadK11) -> PB40B_K11
- U1 pad K4: unconnected-(U1B-PB64B-PadK4) -> PB64B_K4
- U1 pad K5: unconnected-(U1B-PB58A-PadK5) -> PB58A_K5
- U1 pad K6: unconnected-(U1B-PB58B-PadK6) -> PB58B_K6
- U1 pad K7: unconnected-(U1B-PB56A-PadK7) -> PB56A_K7
- U1 pad K8: unconnected-(U1B-PB52B-PadK8) -> PB52B_K8
- U1 pad K9: unconnected-(U1B-PB50B-PadK9) -> PB50B_K9
- U1 pad L1: unconnected-(U1B-PB70B-PadL1) -> PB70B_L1
- U1 pad L10: unconnected-(U1B-PB46A-PadL10) -> PB46A_L10
- U1 pad L11: unconnected-(U1B-PB46B-PadL11) -> PB46B_L11
- U1 pad L2: unconnected-(U1B-PB70A-PadL2) -> PB70A_L2
- U1 pad L5: unconnected-(U1B-PB62A-PadL5) -> PB62A_L5
- U1 pad L6: unconnected-(U1B-PB62B-PadL6) -> PB62B_L6
- U1 pad L7: unconnected-(U1B-PB56B-PadL7) -> PB56B_L7
- U1 pad L8: unconnected-(U1B-PB52A-PadL8) -> PB52A_L8
- U1 pad L9: unconnected-(U1B-PB50A-PadL9) -> PB50A_L9
Routing:
- net PB56A_K7: track 0.00 -> 16.4 mm, vias 0 -> 1
- net USB_DP1: track 0.00 -> 16.2 mm
- net USB_DM1: track 0.00 -> 16.1 mm, vias 0 -> 2
- net PB56B_L7: track 0.00 -> 14.4 mm, vias 0 -> 1
- net PB52A_L8: track 0.00 -> 14.4 mm, vias 0 -> 1
- net FLASH_CLK: track 0.00 -> 14.3 mm
- net FLASH_MOSI: track 0.00 -> 13.9 mm, vias 0 -> 1
- net PB50A_L9: track 0.00 -> 13.2 mm
- net PB52B_K8: track 0.00 -> 12.7 mm, vias 0 -> 1
- net FLASH_D3: track 0.00 -> 12.1 mm
- net PB50B_K9: track 0.00 -> 11.6 mm, vias 0 -> 1
- net JTAG_TMS: track 0.00 -> 9.85 mm
- net PB20A_G10: track 0.00 -> 9.40 mm, vias 0 -> 1
- net PB20B_G11: track 0.00 -> 7.90 mm
- net JTAG_TDI: track 0.00 -> 7.53 mm, vias 0 -> 2
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
Commit message: breakout
Parts:
- removed C17, C66: 10u, Capacitor_SMD:C_0603_1608Metric_Pad1.08x0.95mm_HandSolder
- removed C52, C67: 0.1u, Capacitor_SMD:C_0402_1005Metric_Pad0.74x0.62mm_HandSolder
- removed C53, C54: 0.01u, Capacitor_SMD:C_0402_1005Metric_Pad0.74x0.62mm_HandSolder
- removed C56: 22n, Passive_Robotech:1608-C
- removed FB8: 120Ohm, Inductor_SMD:L_0603_1608Metric_Pad1.05x0.95mm_HandSolder
- removed J2: Conn_01x06, Connector_PinHeader_2.54mm:PinHeader_1x06_P2.54mm_Vertical
- removed LED1: ~, Diode_Robotech:WS2812C-2020
- removed R44: 2.49k, Resistor_SMD:R_0402_1005Metric_Pad0.72x0.64mm_HandSolder
- removed R45: 1.96k, Resistor_SMD:R_0402_1005Metric_Pad0.72x0.64mm_HandSolder
- removed R46: 4.87k, Resistor_SMD:R_0402_1005Metric_Pad0.72x0.64mm_HandSolder
- removed R47: 10k, Resistor_SMD:R_0402_1005Metric_Pad0.72x0.64mm_HandSolder
- removed R48, R49, R50, R53: 49.9, Passive_Robotech:2012-R
- removed R52: 2.2k, Resistor_SMD:R_0402_1005Metric_Pad0.72x0.64mm_HandSolder
- removed U10: DP83822, IC_Robotech:DP83822
- added G***: LOGO, LSM6DSV16XTR:RoboTech_Logo, F.Cu at (118.9, 118.9)
- added H1: MountingHole, MountingHole:MountingHole_3.2mm_M3, F.Cu at (127.5, 107.5)
- added H2: MountingHole, MountingHole:MountingHole_3.2mm_M3, F.Cu at (127.5, 141.5)
- added H3: MountingHole, MountingHole:MountingHole_3.2mm_M3, F.Cu at (144.7, 141.2)
- C48: moved to B.Cu
- D7, R24, R25: moved to F.Cu
- J4: value RJLD260TC1 -> Conn_ARM_JTAG_SWD_10; footprint Connector_Robotech:RJLD260TC1 -> Connector_PinHeader_1.27mm:PinHeader_2x05_P1.27mm_Vertical
- SW2: footprint Button_Switch_THT:SW_Slide-03_Wuerth-WS-SLTV_10x2.5x6.4_P2.54mm -> Button_Switch_SMD:SW_SPDT_PCM12
- moved J4 98.2 mm to (117.5, 142.2), turned to 90 degrees
- moved R10 41.0 mm to (97.0, 125.5), turned to 90 degrees
- moved R7 40.6 mm to (97.0, 131.9), turned to 90 degrees
- moved SW2 39.2 mm to (93.8, 128.7), turned to -90 degrees
- moved SW1 33.8 mm to (116.0, 108.2), turned to -90 degrees
- moved CON1 31.2 mm to (93.5, 110.8), turned to 180 degrees
- moved J3 30.6 mm to (96.0, 140.8), turned to 0 degrees
- moved R20 29.3 mm to (116.8, 111.5), turned to 0 degrees
- moved C46 28.9 mm to (103.6, 142.8), turned to 180 degrees
- moved C1 28.8 mm to (97.3, 109.3), turned to -90 degrees
- moved R15 28.8 mm to (110.5, 108.3)
- moved R41 28.8 mm to (108.1, 108.3)
- moved U8 28.8 mm to (110.5, 110.3)
- moved C63 28.8 mm to (108.0, 111.2)
- moved C64 28.8 mm to (113.0, 109.7)
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Connections:
- D1 pad 2: +3V3 -> +1V8
- D2 pad 2: +3V3 -> +1V8
- D3 pad 2: +3V3 -> +1V8
- D4 pad 2: +3V3 -> +1V8
- J1 pad 10: PB46B_L11 -> PB42A_J8
- J1 pad 11: PB40A_K10 -> PB50B_K9
- J1 pad 12: PB40B_K11 -> PB30B_F7
- J1 pad 13: PB42A_J8 -> PB50A_L9
- J1 pad 14: PB42B_J7 -> PR30A_E7
- J1 pad 15: PB48A_J10 -> PB46A_L10
- J1 pad 16: PB48B_J11 -> PB54A_G9
- J1 pad 17: PB44A_H11 -> PB46B_L11
- J1 pad 18: PB44B_H10 -> PB54B_G8
- J1 pad 19: PB54A_G9 -> PB40A_K10
- J1 pad 20: PB54B_G8 -> PB26A_F8
- J1 pad 21: PB22A_H7 -> PB40B_K11
- J1 pad 22: PB22B_G7 -> PB26B_F9
- J1 pad 23: PB20A_G10 -> PB48A_J10
- J1 pad 24: PB20B_G11 -> unconnected-(J1-Pin_24-Pad24)
- J1 pad 25: PB26A_F8 -> PB48B_J11
- J1 pad 26: PB26B_F9 -> unconnected-(J1-Pin_26-Pad26)
- J1 pad 27: PR30A_E7 -> PB44B_H10
- J1 pad 28: PB30B_F7 -> unconnected-(J1-Pin_28-Pad28)
- J1 pad 29: unconnected-(J1-Pin_29-Pad29) -> PB44A_H11
- J1 pad 30: PR65B_D8 -> unconnected-(J1-Pin_30-Pad30)
- J1 pad 31: PB18A_F11 -> PB20A_G10
- J1 pad 32: PB18B_F10 -> unconnected-(J1-Pin_32-Pad32)
- J1 pad 33: PB16A_E11 -> PB20B_G11
- J1 pad 34: PB16B_E10 -> PR65B_D8
- J1 pad 35: unconnected-(J1-Pin_35-Pad35) -> PB18B_F10
- J1 pad 36: unconnected-(J1-Pin_36-Pad36) -> PB16B_E10
- J1 pad 37: unconnected-(J1-Pin_37-Pad37) -> PB18A_F11
- J1 pad 38: unconnected-(J1-Pin_38-Pad38) -> PB16A_E11
- J1 pad 4: PB56B_L7 -> PB22A_H7
- J1 pad 5: PB52A_L8 -> PB56B_L7
- J1 pad 6: PB52B_K8 -> PB22B_G7
- J1 pad 7: PB50A_L9 -> PB52B_K8
- J1 pad 8: PB50B_K9 -> PB42B_J7
- J1 pad 9: PB46A_L10 -> PB52A_L8
- J4 pad 1: Net-(J4-TD+) -> +3V3
- J4 pad 2: Net-(J4-TD-) -> JTAG_TMS
- J4 pad 3: Net-(J4-RD+) -> GND
- J4 pad 4: Net-(J4-RXCT) -> JTAG_TCK
- J4 pad 5: Net-(J4-RXCT) -> GND
- J4 pad 6: Net-(J4-RD-) -> JTAG_TDO
- J4 pad 8: POWERGND -> JTAG_TDI
- J4 pad 9: unconnected-(J4-GRNA-Pad9) -> GND
- J5 pad 10: +5V -> PB58B_K6
- J5 pad 11: PB70A_L2 -> PB66A_H4
- J5 pad 12: PB70B_L1 -> PB58A_K5
- J5 pad 13: PB62A_L5 -> ADC_DP1_H2
- J5 pad 14: PB62B_L6 -> PB70A_L2
- J5 pad 15: PB64A_J5 -> ADC_DP0_H1
- J5 pad 16: PB64B_K4 -> PB70B_L1
- J5 pad 17: PB68A_J1 -> ADC_DN1_H1
- J5 pad 19: PB66A_H4 -> ADC_DN0_H2
- J5 pad 20: PB66B_J4 -> PB68A_J1
- J5 pad 21: PB60A_G5 -> PB60B_H5
- J5 pad 22: PB60B_H5 -> PR13B_F1
- J5 pad 23: PB58A_K5 -> PB60A_G5
- J5 pad 24: PB58B_K6 -> PR13A_E3
- J5 pad 25: PB24A_F6 -> PR28B_E5
- J5 pad 26: PB24B_F5 -> PR11B_E1
- J5 pad 28: PR28B_E5 -> PR11A_E2
- J5 pad 29: PT67A_B3 -> PT67B_C3
- J5 pad 3: +1V -> unconnected-(J5-Pin_3-Pad3)
- J5 pad 30: PT67B_C3 -> PR7B_C2
- J5 pad 31: PR13A_E3 -> PT67A_B3
- J5 pad 32: PR13B_F1 -> PR7A_B2
- J5 pad 33: PR11A_E2 -> +1V8
- J5 pad 34: PR11B_E1 -> +1V8
- J5 pad 35: unconnected-(J5-Pin_35-Pad35) -> +3V3
- J5 pad 36: PR9B_D1 -> +3V3
- J5 pad 37: PR7A_B2 -> +5V
- J5 pad 38: PR7B_C2 -> +5V
- J5 pad 4: +1V -> unconnected-(J5-Pin_4-Pad4)
- J5 pad 5: +1V8 -> PB64A_J5
- J5 pad 6: +1V8 -> PB62B_L6
- J5 pad 7: +3V3 -> PB64B_K4
- J5 pad 8: +3V3 -> PB62A_L5
- J5 pad 9: +5V -> PB66B_J4
- R16 pad 2: LED1 -> PB44A_H11
- R17 pad 2: LED2 -> PB44B_H10
- R18 pad 2: LED3 -> PB48B_J11
- R19 pad 2: LED4 -> PB48A_J10
- R20 pad 1: SW1 -> PR65B_D8
- R20 pad 2: +3V3 -> +1V8
- SW1 pad 2: SW1 -> PR65B_D8
- U1 pad G1: unconnected-(U1A-ADC_DN0-PadG1) -> ADC_DN0_H2
- U1 pad G2: unconnected-(U1A-ADC_DN1-PadG2) -> ADC_DN1_H1
- U1 pad H1: unconnected-(U1B-ADC_DP0-PadH1) -> ADC_DP0_H1
- U1 pad H2: unconnected-(U1B-ADC_DP1-PadH2) -> ADC_DP1_H2
Routing:
- net +3V3: track 14.7 -> 125.9 mm, vias 2 -> 13
- net +1V8: track 5.89 -> 83.5 mm, vias 6 -> 9
- net GND: track 19.4 -> 71.1 mm, vias 36 -> 79
- net +1V: track 1.06 -> 23.9 mm, vias 3 -> 6
- net JTAG_TDI: track 7.53 -> 24.6 mm, vias 2 -> 3
- net JTAG_TCK: track 5.59 -> 22.6 mm, vias 0 -> 1
- net PR65B_D8: track 2.23 -> 18.9 mm, vias 0 -> 2
- net JTAG_TDO: track 7.49 -> 23.2 mm, vias 2 -> 3
- net PB62B_L6: track 0.35 -> 15.2 mm, vias 0 -> 1
- net USB_DP1: track 16.2 -> 30.7 mm, vias 0 -> 2
- net PB58B_K6: track 0.95 -> 15.4 mm, vias 0 -> 3
- net PB44B_H10: track 0.00 -> 14.4 mm, vias 0 -> 2
- net PB44A_H11: track 0.00 -> 14.3 mm, vias 0 -> 2
- net PB48A_J10: track 0.00 -> 14.2 mm, vias 0 -> 2
- net PB62A_L5: track 0.35 -> 14.3 mm, vias 0 -> 1
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- added copper zone on B.Cu, net GND
- added copper zone on F.Cu, net GND
- added copper zone on In1.Cu, net GND
- added copper zone on In2.Cu, net GND
Other:
- board text added: "CertusNX Core"
- board text added: "ver 1.0"

Commit message: 配置変更
Parts:
- added H4: MountingHole, MountingHole:MountingHole_3.2mm_M3, F.Cu at (93.5, 107.5)
- added Q1: Q_NMOS, Package_TO_SOT_SMD:SOT-416, F.Cu at (110.2, 127.5)
- J1, J5: footprint Connector_Molex:Molex_SlimStack_52991-0408_2x20_P0.50mm_Vertical -> Local:Molex_SlimStack_52991-0408_2x20_P0.50mm_Vertical
- R1, R16, R17, R18, R19, R2, R30, R31, R32, R33, R8, R9: moved to B.Cu
- U9: footprint Package_DFN_QFN:Texas_B3QFN-14-1EP_5x5.5mm_P0.65mm_ThermalVia -> Local:Texas_B3QFN-14-1EP_5x5.5mm_P0.65mm_ThermalVia
- moved H3 51.2 mm to (93.5, 141.5)
- moved L1 12.5 mm to (113.9, 118.7), turned to 0 degrees
- moved R10 12.4 mm to (97.2, 113.0)
- moved R7 12.4 mm to (97.1, 119.5)
- moved SW2 12.4 mm to (93.9, 116.3)
- moved U4 11.5 mm to (99.8, 140.2), turned to -90 degrees
- moved C60 11.0 mm to (114.2, 115.1), turned to 90 degrees
- moved C65 11.0 mm to (108.1, 119.8), turned to 0 degrees
- moved R29 10.5 mm to (108.3, 124.9), turned to -90 degrees
- moved R30 10.3 mm to (108.3, 124.9), turned to -90 degrees
- moved C34 10.0 mm to (99.8, 138.4), turned to 0 degrees
- moved D7 9.11 mm to (94.9, 125.7), turned to 180 degrees
- moved C61 9.08 mm to (102.9, 122.0)
- moved C62 9.08 mm to (104.4, 127.0)
- moved L2 9.08 mm to (100.8, 126.7)
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Connections:
- R29 pad 2: unconnected-(R29-Pad2) -> Net-(Q1-D)
- R30 pad 2: unconnected-(R30-Pad2) -> Net-(Q1-G)
Routing:
- net +5V: track 11.1 -> 39.7 mm, vias 7 -> 1
- net +1V8: track 83.5 -> 63.5 mm
- net ~{PROGRAM}: track 3.36 -> 17.0 mm, vias 0 -> 1
- net USB_DP1: track 30.7 -> 18.2 mm
- net USB_DM1: track 28.1 -> 16.3 mm
- net DONE: track 7.18 -> 18.5 mm, vias 0 -> 1
- net ~{INIT}: track 14.6 -> 20.3 mm, vias 2 -> 1
- net Net-(U4-D+): track 6.00 -> 10.7 mm
- net Net-(U4-D-): track 7.81 -> 12.3 mm
- net Net-(D7-PadA): track 9.06 -> 13.2 mm
- net Net-(Q1-G): track 0.00 -> 3.59 mm, vias 0 -> 1
- net Net-(Q1-D): track 0.00 -> 2.52 mm
- net GND: track 71.1 -> 73.5 mm, vias 79 -> 81
- net +3V3: track 125.9 -> 123.9 mm, vias 13 -> 17
- net +1V8_{AUX}: track 15.0 -> 17.0 mm, vias 4 -> 5
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