File: CertusNX.kicad_sch (KiCad schematic)
At the start: 147 parts, among them J1 USB_C_Receptacle, J2 Conn_01x06, J3 RJLD260TC1, J4 RJLD260TC1, J5 Conn_02x10_Odd_Even, J6 Conn_02x10_Odd_Even, SW1 SW_Push, SW2 SW_SPDT, U1 LFD2NX-17-7MG121I, U10 DP83822, U2 FT232H, U3 W25Q128JVP, U4 FSUSB42MUX, U5 DP83822, U6 TLV62569ADRL, U7 TLV62569ADRL, U8 TLV62569ADRL, U9 TPSM53604RDA, Y1 SiT8008xx-7x-xxN

Commit message: 配置(あきらめ)
Parts:
- removed C49, C57: 0.1u, Passive_Robotech:1608-C, symbol Device:C
- removed C50, C51: 0.01u, Passive_Robotech:1608-C, symbol Device:C
- removed C55: 22n, Passive_Robotech:1608-C, symbol Device:C
- removed C58: 10u, Passive_Robotech:2012-C, symbol Device:C
- removed FB7: 120Ohm, Inductor_SMD:L_0603_1608Metric_Pad1.05x0.95mm_HandSolder, symbol Device:FerriteBead
- removed J1: USB_C_Receptacle, Connector_USB:USB_C_Receptacle_Molex_105450-0101, symbol Connector:USB_C_Receptacle
- removed J3: RJLD260TC1, Connector_Robotech:RJLD260TC1, symbol Connector_Robotech:RJLD260TC1
- removed J5, J6: Conn_02x10_Odd_Even, Connector_Molex:Molex_SlimStack_52991-0208_2x10_P0.50mm_Vertical, symbol Connector_Generic:Conn_02x10_Odd_Even
- removed R21: 10k, Passive_Robotech:2012-R, symbol Device:R
- removed R34: 1.96k, Passive_Robotech:2012-R, symbol Device:R
- removed R35: 2.49k, Passive_Robotech:2012-R, symbol Device:R
- removed R36: 4.87k, Passive_Robotech:2012-R, symbol Device:R
- removed R37, R38, R39, R40: 49.9, Passive_Robotech:2012-R, symbol Device:R
- removed R51: 2.2k, Passive_Robotech:2012-R, symbol Device:R
- removed U5: DP83822, IC_Robotech:DP83822, symbol IC_Robotech:DP83822
- added J1, J5: Conn_02x30_Odd_Even, Connector_Molex:Molex_SlimStack_52991-0608_2x30_P0.50mm_Vertical, symbol Connector_Generic:Conn_02x30_Odd_Even
- added J3: USB_C_Receptacle_USB2.0_16P, Connector_USB:USB_C_Receptacle_GCT_USB4105-xx-A_16P_TopMnt_Horizontal, symbol Connector:USB_C_Receptacle_USB2.0_16P
- C52, C53, C54, C67: footprint Passive_Robotech:1608-C -> Capacitor_SMD:C_0402_1005Metric_Pad0.74x0.62mm_HandSolder
- C59, C60, C61, C62, C63, C64, C65, C66: footprint Passive_Robotech:2012-C -> Capacitor_SMD:C_0603_1608Metric_Pad1.08x0.95mm_HandSolder
- L1, L2, L3: footprint (none) -> Inductor_SMD:L_1210_3225Metric_Pad1.42x2.65mm_HandSolder
- R44, R45, R46, R47, R52: footprint Passive_Robotech:2012-R -> Resistor_SMD:R_0402_1005Metric_Pad0.72x0.64mm_HandSolder
- U2: footprint Package_QFP:LQFP-48_7x7mm_P0.5mm -> Package_DFN_QFN:QFN-48-1EP_8x8mm_P0.5mm_EP6.2x6.2mm
- U4: footprint Package_SO:MSOP-10_3x3mm_P0.5mm -> Local:FSUSB42UMX
Connections:
- net GND: now also J3.A1 (GND), J3.A12 (GND), J3.B1 (GND), J3.B12 (GND), J3.S1 (SHIELD)
- net at R22.1: now also J3.A7 (D-), J3.B7 (D-)
- net at R25.1: now also J3.B5 (CC2)
- net at R23.1: now also J3.A6 (D+), J3.B6 (D+)
- net at R24.1: now also J3.A5 (CC1)
- net at D7.A: now also J3.A4 (VBUS), J3.A9 (VBUS), J3.B4 (VBUS), J3.B9 (VBUS)
- no-connect marks 53 -> 34

Commit message: pin仮
Parts:
- C11, C13, C14, C16, C19, C20, C21, C22, C24, C25, C27, C28, C29, C33, C47: footprint Capacitor_SMD:C_0402_1005Metric_Pad0.74x0.62mm_HandSolder -> Capacitor_SMD:C_0201_0603Metric
- J1, J5: value Conn_02x30_Odd_Even -> Conn_02x20_Odd_Even; footprint Connector_Molex:Molex_SlimStack_52991-0608_2x30_P0.50mm_Vertical -> Connector_Molex:Molex_SlimStack_52991-0408_2x20_P0.50mm_Vertical; symbol Connector_Generic:Conn_02x30_Odd_Even -> Connector_Generic:Conn_02x20_Odd_Even
Connections:
- net +1V: now also J5.3 (Pin_3), J5.4 (Pin_4)
- net +1V8: now also J5.5 (Pin_5), J5.6 (Pin_6)
- net +3V3: now also J5.7 (Pin_7), J5.8 (Pin_8)
- net +5V: now also J5.10 (Pin_10), J5.9 (Pin_9)
- net GND: now also J1.1 (Pin_1), J1.2 (Pin_2), J1.39 (Pin_39), J1.40 (Pin_40), J5.1 (Pin_1), J5.2 (Pin_2), J5.39 (Pin_39), J5.40 (Pin_40)
- net PR7A_B2: now reaches U1.B2 (PR7A)
- net PR7A_B2: now also J5.37 (Pin_37)
- net PT67A_B3: now reaches U1.B3 (PT67A)
- net PT67A_B3: now also J5.29 (Pin_29)
- net PR7B_C2: now reaches U1.C2 (PR7B)
- net PR7B_C2: now also J5.38 (Pin_38)
- net PT67B_C3: now reaches U1.C3 (PT67B)
- net PT67B_C3: now also J5.30 (Pin_30)
- net PR9B_D1: now reaches U1.D1 (PR9B)
- net PR9B_D1: now also J5.36 (Pin_36)
- net PR65B_D8: now reaches U1.D8 (PT65B)
- net PR65B_D8: now also J1.30 (Pin_30)
- net PR11B_E1: now reaches U1.E1 (PR11B)
- net PR11B_E1: now also J5.34 (Pin_34)
- net PR11A_E2: now reaches U1.E2 (PR11A)
- net PR11A_E2: now also J5.33 (Pin_33)
- net PR13A_E3: now reaches U1.E3 (PR13A)
- net PR13A_E3: now also J5.31 (Pin_31)
- net PR28B_E5: now reaches U1.E5 (PB28B)
- net PR28B_E5: now also J5.28 (Pin_28)
- net PR28A_E6: now reaches U1.E6 (PB28A)
- net PR28A_E6: now also J5.27 (Pin_27)
- net PR30A_E7: now reaches U1.E7 (PB30A)
- net PR30A_E7: now also J1.27 (Pin_27)
- net PR13B_F1: now reaches U1.F1 (PR13B)
- net PR13B_F1: now also J5.32 (Pin_32)
- net PB24B_F5: now reaches U1.F5 (PB24B)
- net PB24B_F5: now also J5.26 (Pin_26)
- net PB24A_F6: now reaches U1.F6 (PB24A)
- net PB24A_F6: now also J5.25 (Pin_25)
- net PB30B_F7: now reaches U1.F7 (PB30B)
- net PB30B_F7: now also J1.28 (Pin_28)
- net PB26A_F8: now reaches U1.F8 (PB26A)
- net PB26A_F8: now also J1.25 (Pin_25)
- net PB26B_F9: now reaches U1.F9 (PB26B)
- net PB26B_F9: now also J1.26 (Pin_26)
- net PB60A_G5: now reaches U1.G5 (PB60A)
- net PB60A_G5: now also J5.21 (Pin_21)
- net PB22B_G7: now reaches U1.G7 (PB22B)
- net PB22B_G7: now also J1.22 (Pin_22)
- net PB16B_E10: now reaches U1.E10 (PB16B)
- net PB16B_E10: now also J1.34 (Pin_34)
- net PB16A_E11: now reaches U1.E11 (PB16A)
- net PB16A_E11: now also J1.33 (Pin_33)
- net PB18B_F10: now reaches U1.F10 (PB18B)
- net PB18B_F10: now also J1.32 (Pin_32)
- net PB18A_F11: now reaches U1.F11 (PB18A)
- net PB18A_F11: now also J1.31 (Pin_31)
- net PB20A_G10: now reaches U1.G10 (PB20A)
- net PB20A_G10: now also J1.23 (Pin_23)
- net PB20B_G11: now reaches U1.G11 (PB20B)
- net PB20B_G11: now also J1.24 (Pin_24)
- net PB54B_G8: now reaches U1.G8 (PB54B)
- net PB54B_G8: now also J1.20 (Pin_20)
- net PB54A_G9: now reaches U1.G9 (PB54A)
- net PB54A_G9: now also J1.19 (Pin_19)
- net PB44B_H10: now reaches U1.H10 (PB44B)
- net PB44B_H10: now also J1.16 (Pin_16)
- net PB44A_H11: now reaches U1.H11 (PB44A)
- net PB44A_H11: now also J1.15 (Pin_15)
- net PB66A_H4: now reaches U1.H4 (PB66A)
- net PB66A_H4: now also J5.19 (Pin_19)
- net PB60B_H5: now reaches U1.H5 (PB60B)
- net PB60B_H5: now also J5.22 (Pin_22)
- net PB22A_H7: now reaches U1.H7 (PB22A)
- net PB22A_H7: now also J1.21 (Pin_21)
- net PB68A_J1: now reaches U1.J1 (PB68A)
- net PB68A_J1: now also J5.17 (Pin_17)
- net PB48A_J10: now reaches U1.J10 (PB48A)
- net PB48A_J10: now also J1.13 (Pin_13)
- net PB48B_J11: now reaches U1.J11 (PB48B)
- net PB48B_J11: now also J1.14 (Pin_14)
- net PB68B_J2: now reaches U1.J2 (PB68B)
- net PB68B_J2: now also J5.18 (Pin_18)
- net PB66B_J4: now reaches U1.J4 (PB66B)
- net PB66B_J4: now also J5.20 (Pin_20)
- net PB64A_J5: now reaches U1.J5 (PB64A)
- net PB64A_J5: now also J5.15 (Pin_15)
- net PB42B_J7: now reaches U1.J7 (PB42B)
- net PB42B_J7: now also J1.12 (Pin_12)
- net PB42A_J8: now reaches U1.J8 (PB42A)
- net PB42A_J8: now also J1.11 (Pin_11)
- net PB40A_K10: now reaches U1.K10 (PB40A)
- net PB40A_K10: now also J1.9 (Pin_9)
- net PB40B_K11: now reaches U1.K11 (PB40B)
- net PB40B_K11: now also J1.10 (Pin_10)
- net PB64B_K4: now reaches U1.K4 (PB64B)
- net PB64B_K4: now also J5.16 (Pin_16)
- net PB58A_K5: now reaches U1.K5 (PB58A)
- net PB58A_K5: now also J5.23 (Pin_23)
- net PB58B_K6: now reaches U1.K6 (PB58B)
- net PB58B_K6: now also J5.24 (Pin_24)
- net PB56A_K7: now reaches U1.K7 (PB56A)
- net PB56A_K7: now also J1.3 (Pin_3)
- net PB52B_K8: now reaches U1.K8 (PB52B)
- net PB52B_K8: now also J1.6 (Pin_6)
- net PB50B_K9: now reaches U1.K9 (PB50B)
- net PB50B_K9: now also J1.18 (Pin_18)
- net PB70B_L1: now reaches U1.L1 (PB70B)
- net PB70B_L1: now also J5.12 (Pin_12)
- net PB46A_L10: now reaches U1.L10 (PB46A)
- net PB46A_L10: now also J1.7 (Pin_7)
- net PB46B_L11: now reaches U1.L11 (PB46B)
- net PB46B_L11: now also J1.8 (Pin_8)
- net PB70A_L2: now reaches U1.L2 (PB70A)
- net PB70A_L2: now also J5.11 (Pin_11)
- net PB62A_L5: now reaches U1.L5 (PB62A)
- net PB62A_L5: now also J5.13 (Pin_13)
- net PB62B_L6: now reaches U1.L6 (PB62B)
- net PB62B_L6: now also J5.14 (Pin_14)
- net PB56B_L7: now reaches U1.L7 (PB56B)
- net PB56B_L7: now also J1.4 (Pin_4)
- net PB52A_L8: now reaches U1.L8 (PB52A)
- net PB52A_L8: now also J1.5 (Pin_5)
- net PB50A_L9: now reaches U1.L9 (PB50A)
- net PB50A_L9: now also J1.17 (Pin_17)

Commit message: breakout
Parts:
- removed C17, C66: 10u, Capacitor_SMD:C_0603_1608Metric_Pad1.08x0.95mm_HandSolder, symbol Device:C
- removed C52, C67: 0.1u, Capacitor_SMD:C_0402_1005Metric_Pad0.74x0.62mm_HandSolder, symbol Device:C
- removed C53, C54: 0.01u, Capacitor_SMD:C_0402_1005Metric_Pad0.74x0.62mm_HandSolder, symbol Device:C
- removed C56: 22n, Passive_Robotech:1608-C, symbol Device:C
- removed FB8: 120Ohm, Inductor_SMD:L_0603_1608Metric_Pad1.05x0.95mm_HandSolder, symbol Device:FerriteBead
- removed J2: Conn_01x06, Connector_PinHeader_2.54mm:PinHeader_1x06_P2.54mm_Vertical, symbol Connector_Generic:Conn_01x06
- removed J4: RJLD260TC1, Connector_Robotech:RJLD260TC1, symbol Connector_Robotech:RJLD260TC1
- removed LED1: ~, Diode_Robotech:WS2812C-2020, symbol Diode_Robotech:WS2812C
- removed R44: 2.49k, Resistor_SMD:R_0402_1005Metric_Pad0.72x0.64mm_HandSolder, symbol Device:R
- removed R45: 1.96k, Resistor_SMD:R_0402_1005Metric_Pad0.72x0.64mm_HandSolder, symbol Device:R
- removed R46: 4.87k, Resistor_SMD:R_0402_1005Metric_Pad0.72x0.64mm_HandSolder, symbol Device:R
- removed R47: 10k, Resistor_SMD:R_0402_1005Metric_Pad0.72x0.64mm_HandSolder, symbol Device:R
- removed R48, R49, R50, R53: 49.9, Passive_Robotech:2012-R, symbol Device:R
- removed R52: 2.2k, Resistor_SMD:R_0402_1005Metric_Pad0.72x0.64mm_HandSolder, symbol Device:R
- removed U10: DP83822, IC_Robotech:DP83822, symbol IC_Robotech:DP83822
- added H1, H2, H3: MountingHole, MountingHole:MountingHole_3.2mm_M3, symbol Mechanical:MountingHole
- added J4: Conn_ARM_JTAG_SWD_10, Connector_PinHeader_1.27mm:PinHeader_2x05_P1.27mm_Vertical, symbol Connector:Conn_ARM_JTAG_SWD_10
- SW2: footprint Button_Switch_THT:SW_Slide-03_Wuerth-WS-SLTV_10x2.5x6.4_P2.54mm -> Button_Switch_SMD:SW_SPDT_PCM12
Connections:
- net LED1 is gone; now on net PB44A_H11: R16.2
- net LED2 is gone; now on net PB44B_H10: R17.2
- net LED3 is gone; now on net PB48B_J11: R18.2
- net LED4 is gone; now on net PB48A_J10: R19.2
- net SW1 is gone; now on net PR65B_D8: R20.1, SW1.2
- net +1V: no longer J5.3 (Pin_3), J5.4 (Pin_4)
- net +1V8: now also D1.2 (A), D2.2 (A), D3.2 (A), D4.2 (A), J5.33 (Pin_33), J5.34 (Pin_34), R20.2; no longer J5.5 (Pin_5), J5.6 (Pin_6)
- net +3V3: now also J5.35 (Pin_35), J5.36 (Pin_36), J4.1 (VTref); no longer D1.2 (A), D2.2 (A), D3.2 (A), D4.2 (A), J5.7 (Pin_7), J5.8 (Pin_8), R20.2
- net +5V: now also J5.37 (Pin_37), J5.38 (Pin_38); no longer J5.10 (Pin_10), J5.9 (Pin_9)
- net GND: now also J4.3 (GND), J4.5 (GND), J4.9 (GNDDetect)
- net JTAG_TCK: now also J4.4 (SWCLK/TCK)
- net JTAG_TDI: now also J4.8 (NC/TDI)
- net JTAG_TDO: now also J4.6 (SWO/TDO)
- net JTAG_TMS: now also J4.2 (SWDIO/TMS)
- net PB16A_E11: now also J1.38 (Pin_38); no longer J1.33 (Pin_33)
- net PB16B_E10: now also J1.36 (Pin_36); no longer J1.34 (Pin_34)
- net PB18A_F11: now also J1.37 (Pin_37); no longer J1.31 (Pin_31)
- net PB18B_F10: now also J1.35 (Pin_35); no longer J1.32 (Pin_32)
- net PB20A_G10: now also J1.31 (Pin_31); no longer J1.23 (Pin_23)
- net PB20B_G11: now also J1.33 (Pin_33); no longer J1.24 (Pin_24)
- net PB22A_H7: now also J1.4 (Pin_4); no longer J1.21 (Pin_21)
- net PB22B_G7: now also J1.6 (Pin_6); no longer J1.22 (Pin_22)
- net PB24A_F6: no longer J5.25 (Pin_25)
- net PB24B_F5: no longer J5.26 (Pin_26)
- net PB26A_F8: now also J1.20 (Pin_20); no longer J1.25 (Pin_25)
- net PB26B_F9: now also J1.22 (Pin_22); no longer J1.26 (Pin_26)
- net PB30B_F7: now also J1.12 (Pin_12); no longer J1.28 (Pin_28)
- net PB40A_K10: now also J1.19 (Pin_19); no longer J1.9 (Pin_9)
- net PB40B_K11: now also J1.21 (Pin_21); no longer J1.10 (Pin_10)
- net PB42A_J8: now also J1.10 (Pin_10); no longer J1.11 (Pin_11)
- net PB42B_J7: now also J1.8 (Pin_8); no longer J1.12 (Pin_12)
- net PB44A_H11: now also J1.29 (Pin_29); no longer J1.15 (Pin_15)
- net PB44B_H10: now also J1.27 (Pin_27); no longer J1.16 (Pin_16)
- net PB46A_L10: now also J1.15 (Pin_15); no longer J1.7 (Pin_7)
- net PB46B_L11: now also J1.17 (Pin_17); no longer J1.8 (Pin_8)
- net PB48A_J10: now also J1.23 (Pin_23); no longer J1.13 (Pin_13)
- net PB48B_J11: now also J1.25 (Pin_25); no longer J1.14 (Pin_14)
- net PB50A_L9: now also J1.13 (Pin_13); no longer J1.17 (Pin_17)
- net PB50B_K9: now also J1.11 (Pin_11); no longer J1.18 (Pin_18)
- net PB52A_L8: now also J1.9 (Pin_9); no longer J1.5 (Pin_5)
- net PB52B_K8: now also J1.7 (Pin_7); no longer J1.6 (Pin_6)
- net PB54A_G9: now also J1.16 (Pin_16); no longer J1.19 (Pin_19)
- net PB54B_G8: now also J1.18 (Pin_18); no longer J1.20 (Pin_20)
- net PB56B_L7: now also J1.5 (Pin_5); no longer J1.4 (Pin_4)
- net PB58A_K5: now also J5.12 (Pin_12); no longer J5.23 (Pin_23)
- net PB58B_K6: now also J5.10 (Pin_10); no longer J5.24 (Pin_24)
- net PB60A_G5: now also J5.23 (Pin_23); no longer J5.21 (Pin_21)
- net PB60B_H5: now also J5.21 (Pin_21); no longer J5.22 (Pin_22)
- net PB62A_L5: now also J5.8 (Pin_8); no longer J5.13 (Pin_13)
- net PB62B_L6: now also J5.6 (Pin_6); no longer J5.14 (Pin_14)
- net PB64A_J5: now also J5.5 (Pin_5); no longer J5.15 (Pin_15)
- net PB64B_K4: now also J5.7 (Pin_7); no longer J5.16 (Pin_16)
- net PB66A_H4: now also J5.11 (Pin_11); no longer J5.19 (Pin_19)
- net PB66B_J4: now also J5.9 (Pin_9); no longer J5.20 (Pin_20)
- net PB68A_J1: now also J5.20 (Pin_20); no longer J5.17 (Pin_17)
- net PB70A_L2: now also J5.14 (Pin_14); no longer J5.11 (Pin_11)
- net PB70B_L1: now also J5.16 (Pin_16); no longer J5.12 (Pin_12)
- net PR11A_E2: now also J5.28 (Pin_28); no longer J5.33 (Pin_33)
- net PR11B_E1: now also J5.26 (Pin_26); no longer J5.34 (Pin_34)
- net PR13A_E3: now also J5.24 (Pin_24); no longer J5.31 (Pin_31)
- net PR13B_F1: now also J5.22 (Pin_22); no longer J5.32 (Pin_32)
- net PR28B_E5: now also J5.25 (Pin_25); no longer J5.28 (Pin_28)
- net PR30A_E7: now also J1.14 (Pin_14); no longer J1.27 (Pin_27)
- net PR65B_D8: now also J1.34 (Pin_34); no longer J1.30 (Pin_30)
- net PR7A_B2: now also J5.32 (Pin_32); no longer J5.37 (Pin_37)
- net PR7B_C2: now also J5.30 (Pin_30); no longer J5.38 (Pin_38)
- net PR9B_D1: no longer J5.36 (Pin_36)
- net PT67A_B3: now also J5.31 (Pin_31); no longer J5.29 (Pin_29)
- net PT67B_C3: now also J5.29 (Pin_29); no longer J5.30 (Pin_30)
- net ADC_DN0_H2: now reaches U1.G1 (ADC_DN0)
- net ADC_DN0_H2: now also J5.19 (Pin_19)
- net ADC_DN1_H1: now reaches U1.G2 (ADC_DN1)
- net ADC_DN1_H1: now also J5.17 (Pin_17)
- net ADC_DP0_H1: now reaches U1.H1 (ADC_DP0)
- net ADC_DP0_H1: now also J5.15 (Pin_15)
- net ADC_DP1_H2: now reaches U1.H2 (ADC_DP1)
- net ADC_DP1_H2: now also J5.13 (Pin_13)
- no-connect marks 34 -> 22
Other:
- note removed: "RX_D0 to MODE4 COL to MODE1 (->PHY address=2)"

Commit message: 配置変更
Parts:
- added H4: MountingHole, MountingHole:MountingHole_3.2mm_M3, symbol Mechanical:MountingHole
- added Q1: Q_NMOS, Package_TO_SOT_SMD:SOT-416, symbol Device:Q_NMOS
- J1, J5: footprint Connector_Molex:Molex_SlimStack_52991-0408_2x20_P0.50mm_Vertical -> Local:Molex_SlimStack_52991-0408_2x20_P0.50mm_Vertical
- U9: footprint Package_DFN_QFN:Texas_B3QFN-14-1EP_5x5.5mm_P0.65mm_ThermalVia -> Local:Texas_B3QFN-14-1EP_5x5.5mm_P0.65mm_ThermalVia
Connections:
- net GND: now also Q1.S
- net at R30.2: now also Q1.G
- net at R29.2: now also Q1.D
Other:
- moved on the sheet: R30
Changed lines of the file:
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@@
 	(wire
 		(pts
+			(xy 66.04 383.54) (xy 67.31 383.54)
+		)
+		(stroke
+			(width 0)
+			(type default)
+		)
+	)
+	(wire
+		(pts
 			(xy 227.33 265.43) (xy 224.79 265.43)
 		)
@@
 	(wire
 		(pts
+			(xy 74.93 375.92) (xy 74.93 378.46)
+		)
+		(stroke
+			(width 0)
+			(type default)
+		)
+	)
+	(wire
+		(pts
 			(xy 68.58 255.27) (xy 71.12 255.27)
 		)
@@
 	(wire
 		(pts
+			(xy 74.93 389.89) (xy 74.93 388.62)
+		)
+		(stroke
+			(width 0)
+			(type default)
+		)
+	)
+	(wire
+		(pts
 			(xy 68.58 308.61) (xy 71.12 308.61)
 		)
@@
 	(wire
 		(pts
-			(xy 49.53 383.54) (xy 64.77 383.54)
+			(xy 49.53 383.54) (xy 58.42 383.54)
 		)
 		(stroke
@@
 	(symbol
 		(lib_id "power:GND")
-		(at 74.93 388.62 0)
+		(at 74.93 389.89 0)
 		(unit 1)
 		(exclude_from_sim no)
@@
 		(fields_autoplaced yes)
 		(property "Reference" "#PWR076"
-			(at 74.93 394.97 0)
+			(at 74.93 396.24 0)
 			(effects
 				(font
@@
 		)
 		(property "Value" "GND"
-			(at 74.93 393.7 0)
+			(at 74.93 394.97 0)
 			(effects
 				(font
@@
 		)
 		(property "Footprint" ""
-			(at 74.93 388.62 0)
+			(at 74.93 389.89 0)
 			(effects
 				(font
@@
 		)
 		(property "Datasheet" ""
-			(at 74.93 388.62 0)
+			(at 74.93 389.89 0)
 			(effects
 				(font
@@
 		)
 		(property "Description" "Power symbol creates a global label with name \"GND\" , ground"
-			(at 74.93 388.62 0)
+			(at 74.93 389.89 0)
 			(effects
 				(font
@@
 	(symbol
 		(lib_id "Device:R")
-		(at 68.58 383.54 90)
+		(at 62.23 383.54 90)
+		(mirror x)
 		(unit 1)
 		(exclude_from_sim no)
@@
 		(on_board yes)
 		(dnp no)
-		(fields_autoplaced yes)
 		(property "Reference" "R30"
-			(at 68.58 377.19 90)
+			(at 62.23 389.89 90)
 			(effects
 				(font
@@
 		)
 		(property "Value" "1k"
-			(at 68.58 379.73 90)
+			(at 62.23 387.35 90)
 			(effects
 				(font
@@
 		)
 		(property "Footprint" "Resistor_SMD:R_0402_1005Metric_Pad0.72x0.64mm_HandSolder"
-			(at 68.58 385.318 90)
+			(at 62.23 381.762 90)
 			(effects
 				(font
@@
 		)
 		(property "Datasheet" "~"
-			(at 68.58 383.54 0)
+			(at 62.23 383.54 0)
 			(effects
 				(font
@@
 		)
 		(property "Description" "Resistor"
-			(at 68.58 383.54 0)
+			(at 62.23 383.54 0)
 			(effects
 				(font
@@
 			)
 		)
-		(property "Footprint" "Package_DFN_QFN:Texas_B3QFN-14-1EP_5x5.5mm_P0.65mm_ThermalVia"
+		(property "Footprint" "Local:Texas_B3QFN-14-1EP_5x5.5mm_P0.65mm_ThermalVia"
 			(at 68.58 62.23 0)
 			(effects
@@
 			)
 		)
-		(property "Footprint" "Connector_Molex:Molex_SlimStack_52991-0408_2x20_P0.50mm_Vertical"
+		(property "Footprint" "Local:Molex_SlimStack_52991-0408_2x20_P0.50mm_Vertical"
 			(at 384.81 298.45 0)
 			(effects
@@
 	)
 	(symbol
+		(lib_id "Device:Q_NMOS")
+		(at 72.39 383.54 0)
+		(unit 1)
+		(exclude_from_sim no)
+		(in_bom yes)
+		(on_board yes)
+		(dnp no)
+		(fields_autoplaced yes)
+		(property "Reference" "Q1"
+			(at 78.74 382.2699 0)
+			(effects
+				(font
+					(size 1.27 1.27)
+				)
+				(justify left)
+			)
+		)
+		(property "Value" "Q_NMOS"
+			(at 78.74 384.8099 0)
+			(effects
+				(font
+					(size 1.27 1.27)
+				)
+				(justify left)
+			)
+		)
+		(property "Footprint" "Package_TO_SOT_SMD:SOT-416"
+			(at 77.47 381 0)
+			(effects
+				(font
+					(size 1.27 1.27)
+				)
+				(hide yes)
+			)
+		)
+		(property "Datasheet" "~"
+			(at 72.39 383.54 0)
+			(effects
+				(font
+					(size 1.27 1.27)
+				)
+				(hide yes)
+			)
+		)
+		(property "Description" "N-MOSFET transistor"
+			(at 72.39 383.54 0)
+			(effects
+				(font
+					(size 1.27 1.27)
+				)
+				(hide yes)
+			)
+		)
+		(pin "D"
+		)
+		(pin "S"
+		)
+		(pin "G"
+		)
+		(instances
+			(project ""
+				(path "/809f207a-02f3-4831-9f3a-c9960499091a"
+					(reference "Q1")
+					(unit 1)
+				)
+			)
+		)
+	)
+	(symbol
 		(lib_id "power:GND")
 		(at 118.11 54.61 0)
@@
 	)
 	(symbol
+		(lib_id "Mechanical:MountingHole")
+		(at 367.03 165.1 0)
+		(unit 1)
+		(exclude_from_sim no)
+		(in_bom no)
+		(on_board yes)
+		(dnp no)
+		(fields_autoplaced yes)
+		(property "Reference" "H4"
+			(at 369.57 163.8299 0)
+			(effects
+				(font
+					(size 1.27 1.27)
+				)
+				(justify left)
+			)
+		)
+		(property "Value" "MountingHole"
+			(at 369.57 166.3699 0)
+			(effects
+				(font
+					(size 1.27 1.27)
+				)
+				(justify left)
+			)
+		)
+		(property "Footprint" "MountingHole:MountingHole_3.2mm_M3"
+			(at 367.03 165.1 0)
+			(effects
+				(font
+					(size 1.27 1.27)
+				)
+				(hide yes)
+			)
+		)
+		(property "Datasheet" "~"
+			(at 367.03 165.1 0)
+			(effects
+				(font
+					(size 1.27 1.27)
+				)
+				(hide yes)
+			)
+		)
+		(property "Description" "Mounting Hole without connection"
+			(at 367.03 165.1 0)
+			(effects
+				(font
+					(size 1.27 1.27)
+				)
+				(hide yes)
+			)
+		)
+		(instances
+			(project "CertusNX"
+				(path "/809f207a-02f3-4831-9f3a-c9960499091a"
+					(reference "H4")
+					(unit 1)
+				)
+			)
+		)
+	)
+	(symbol
 		(lib_id "Device:C")
 		(at 285.75 251.46 0)
@@
 			)
 		)
-		(property "Footprint" "Connector_Molex:Molex_SlimStack_52991-0408_2x20_P0.50mm_Vertical"
+		(property "Footprint" "Local:Molex_SlimStack_52991-0408_2x20_P0.50mm_Vertical"
 			(at 436.88 298.45 0)
 			(effects
